File: Navitron.brd (EAGLE design)
At the start: 70 x 70 mm, 78 parts, among them J2 DX07S016JA1R1500, Q1 ROHM_RUM002N02T2LROHM_RUM002N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, Q2 2.5A/30V, Q3 ROHM_RUM002N02T2LROHM_RUM002N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, Q4 ROHM_RUM002N02T2LROHM_RUM002N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, Q5 ROHM_RUM002N02T2LROHM_RUM002N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, T1 BC847, T2 BC847, U1 ESP32-WROOM-32, U2 9DoF IMU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

Commit message: Update Navitron.brd
Parts:
- removed R22: 2.2k, SparkFun-Resistors:0402-TIGHT
- R14, R15, R16, R17, R19, R20, R21: device SparkFun-Resistors:0402-TIGHT -> SparkFun-Resistors:0603
- R8: value 470 -> 2.2k; device SparkFun-Resistors:0402-TIGHT -> SparkFun-Resistors:0603
- moved R17 110.5 mm to (-17.0, -39.0)
- moved R15 101.7 mm to (-17.0, -31.0)
- moved R16 100.9 mm to (-17.0, -35.0), turned to 0 degrees
- moved R14 100.8 mm to (-17.0, -27.0), turned to 0 degrees
- moved R8 95.2 mm to (-17.0, -23.0)
- moved R19 41.1 mm to (-17.0, -43.0)
- moved C10 36.0 mm to (11.0, 33.0), turned to 180 degrees
- moved R20 32.0 mm to (-17.0, -47.0)
- moved R21 28.0 mm to (-17.0, -51.0)
- moved RX1 12.2 mm to (49.5, 19.5)
- moved TX1 11.2 mm to (49.5, 17.5)
- moved R9 10.0 mm to (54.5, 21.5)
- moved R18 9.06 mm to (54.5, 19.5)
- moved AP2112K-1.8 7.10 mm to (58.8, 35.5), turned to 90 degrees
- moved C11 7.00 mm to (58.7, 42.6)
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Connections:
- net N$31 renamed TO_RX_LED
- net N$32 renamed TO_TX_LED
- net N$33 renamed TX_RX_LED_SUPPLY
- net N$6 renamed V3_CH340
- net 1.8V: now also R15.2, R17.2, R8.2; no longer R14.2, R16.2, R22.2
- net DI: no longer R8.1
- net FSYNC: now also R17.1; no longer R20.1
- net INT: now also R20.1; no longer R22.1
- net N$10: no longer R8.2
- net N$14: now also R16.2; no longer R15.2
- net N$15: now also R14.2; no longer R17.2
- net SCL: now also R16.1; no longer R15.1
- net SCL1V8: now also R15.1; no longer R14.1
- net SDA: now also R14.1; no longer R17.1
- net SDA1V8: now also R8.1; no longer R16.1
Routing:
- net SDA: track 37.5 -> 0.00 mm, vias 1 -> 0
- net V_USB: track 46.2 -> 80.3 mm
- net SCL: track 32.1 -> 0.50 mm, vias 1 -> 0
- net 3.3V: track 42.1 -> 19.3 mm, vias 3 -> 1
- net DI: track 9.46 -> 0.00 mm
- net N$14: track 6.94 -> 0.00 mm
- net SDA1V8: track 4.77 -> 0.00 mm
- net N$16: track 3.81 -> 0.00 mm
- net N$15: track 3.13 -> 0.06 mm
- net SCL1V8: track 2.71 -> 0.00 mm
- net N$13: track 2.40 -> 0.06 mm
- net N$12: track 2.05 -> 0.00 mm
- net TXO: track 50.5 -> 48.5 mm, vias 3 -> 2
- net TO_TX_LED: track 2.27 -> 4.10 mm
- net TO_RX_LED: track 2.27 -> 4.10 mm
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
Commit message: Update Navitron.brd
Parts:
- moved R21 141.4 mm to (83.0, 49.0)
- moved R14 123.5 mm to (84.0, 44.0)
- moved Q3 118.2 mm to (80.0, 60.0)
- moved Q5 118.2 mm to (80.0, 49.0)
- moved R15 118.2 mm to (79.0, 38.0)
- moved R16 118.2 mm to (79.0, 34.0)
- moved R17 118.2 mm to (79.0, 30.0)
- moved R19 118.2 mm to (79.0, 26.0)
- moved R20 107.8 mm to (53.0, 35.0)
- moved R8 89.8 mm to (54.0, 32.0), turned to 90 degrees
- moved JP5 44.3 mm to (90.1, 39.5), turned to 270 degrees
- moved Q1 14.3 mm to (50.0, 33.0)
- moved Q4 12.5 mm to (56.0, 32.0)
- moved C9 6.57 mm to (59.0, 40.5)
- moved C12 2.00 mm to (59.0, 38.0)
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Routing:
- net SCL: track 0.50 -> 37.0 mm, vias 0 -> 1
- net SDA: track 0.00 -> 33.4 mm, vias 0 -> 1
- net SDA1V8: track 0.00 -> 14.8 mm, vias 0 -> 2
- net SCL1V8: track 0.00 -> 13.5 mm, vias 0 -> 2
- net N$16: track 0.00 -> 8.43 mm, vias 0 -> 2
- net 3.3V: track 19.3 -> 27.0 mm
- net GND: track 63.3 -> 67.5 mm
- net INT: track 0.00 -> 2.39 mm

Commit message: Update Navitron.brd
Parts:
- moved R19 41.2 mm to (47.0, 52.0)
- moved R17 35.5 mm to (49.0, 49.0)
- moved R14 34.5 mm to (54.0, 27.0)
- moved JP5 33.8 mm to (58.1, 28.5), turned to 90 degrees
- moved Q3 33.8 mm to (49.0, 46.5), turned to 180 degrees
- moved R15 29.6 mm to (50.0, 44.0)
- moved Q5 27.3 mm to (53.0, 45.0)
- moved R16 27.3 mm to (52.0, 30.0), turned to 270 degrees
- moved R21 27.3 mm to (56.0, 45.0)
- moved R12 6.40 mm to (50.1, 54.4), turned to 270 degrees
- moved JP3 4.00 mm to (54.4, 47.5)
- moved POWER2 1.00 mm to (52.4, 50.4), turned to 90 degrees
Routing:
- net FSYNC_VIN: track 0.00 -> 19.0 mm, vias 0 -> 2
- net INT_VIN: track 0.00 -> 16.0 mm, vias 0 -> 2
- net FSYNC: track 0.00 -> 14.2 mm, vias 0 -> 2
- net 1.8V: track 0.11 -> 13.8 mm
- net INT: track 2.39 -> 10.0 mm, vias 0 -> 2
- net N$14: track 0.00 -> 6.21 mm
- net SDA: track 33.4 -> 38.4 mm
- net N$15: track 0.00 -> 3.41 mm
- net N$16: track 8.43 -> 11.6 mm
- net N$12: track 0.00 -> 3.19 mm
- net N$13: track 0.06 -> 2.70 mm
- net SCL1V8: track 13.5 -> 15.8 mm
- net SCL: track 37.0 -> 38.2 mm

Commit message: Update
Parts:
- removed S1: RESET, SparkFun-Switches:TACTILE_SWITCH_SMD_4.6X2.8MM
- removed S2: 0, SparkFun-Switches:TACTILE_SWITCH_SMD_4.6X2.8MM
- added U$1, U$2: MYSWITCH, MyLib:MY-BUTTON
Connections:
- net 0: now also U$2.P$2; no longer S2.3, S2.4
- net GND: now also U$1.P$1, U$2.P$1; no longer S1.1, S1.2, S2.1, S2.2
- net RESET: now also U$1.P$2; no longer S1.3, S1.4
Routing:
- net VIN: track 13.3 -> 29.0 mm
- net GND: track 67.5 -> 81.2 mm, vias 10 -> 11
- net 0: track 20.5 -> 15.2 mm
- net 3.3V: track 27.0 -> 30.4 mm
- net INT_VIN: track 16.0 -> 13.4 mm
- net RESET: track 38.4 -> 36.5 mm
- net V_BATT: track 43.9 -> 45.2 mm
- net WS13_14: track 8.46 -> 9.10 mm

Commit message: Inspected
Parts:
- added R22: 470, SparkFun-Resistors:0603
- moved C3 6.40 mm to (11.8, 27.5)
- moved JP3 1.00 mm to (54.4, 48.5)
Connections:
- net DO renamed WS9_10
- net N$16 renamed REGOUT
- net N$2 renamed CHAR_LED_VIN
- net N$3 renamed STAT
- net N$4 renamed TO_T2
- net N$5 renamed TO_T1
- net N$7 renamed PROG
- removed net N$10: WS1.4
- new net DI_TO_WS: R22.1, WS1.4
- net DI: now also R22.2
Routing:
- net 3.3V: track 30.4 -> 52.4 mm, vias 1 -> 6
- net DI_TO_WS: track 0.00 -> 18.0 mm, vias 0 -> 2
- net DI: track 0.00 -> 11.1 mm
- net 1.8V: track 13.9 -> 18.6 mm, vias 0 -> 2
- net GND: track 81.2 -> 78.3 mm
